File: hw/fanctl/fanctl.sch (KiCad schematic (older format))
At the start: 25 parts, among them J1 FAN, J2 Screw_Terminal_01x05, M1 FAN, M2 FAN, Q1 BS170, Q2 BS170, Q3 BS170, Q4 BS170, U1 MCP9700-E

Commit message: schematic drc
Parts:
- removed J2: Screw_Terminal_01x05, symbol Connector:Screw_Terminal_01x05
- added J2: Screw_Terminal_01x06, symbol Connector:Screw_Terminal_01x06
Connections:
- net +12V: now also J2.2 (Pin_2)
- net +3V3: now also J2.3 (Pin_3)
- net GND: now also J2.1 (Pin_1)
- net PWM: now also J2.4 (Pin_4)
- net TACO: now also J2.5 (Pin_5)
- net TEMP: now also J2.6 (Pin_6)
Other:
- moved on the sheet: R5
Changed lines of the file:
@@
 	1    0    0    -1
 $EndComp
-Connection ~ 9200 1650
 $Comp
 L power:GND #PWR07
@@
 L Device:R R5
 U 1 1 60FB1FE4
-P 9200 1500
-F 0 "R5" H 9270 1546 50  0000 L CNN
-F 1 "0" H 9270 1455 50  0000 L CNN
-F 2 "" V 9130 1500 50  0001 C CNN
-F 3 "~" H 9200 1500 50  0001 C CNN
-	1    9200 1500
-	1    0    0    -1
-$EndComp
-Wire Wire Line
-	9200 1350 9200 1250
+P 9200 1450
+F 0 "R5" H 9270 1496 50  0000 L CNN
+F 1 "0" H 9270 1405 50  0000 L CNN
+F 2 "" V 9130 1450 50  0001 C CNN
+F 3 "~" H 9200 1450 50  0001 C CNN
+	1    9200 1450
+	1    0    0    -1
+$EndComp
 Text Notes 7550 600  0    50   ~ 0
 Adjust RC values to filter digital noise
@@
 	1    0    0    -1
 $EndComp
+Text Label 1800 4250 0    50   ~ 0
+TACO
 Text Label 1800 4350 0    50   ~ 0
-TACO
-Text Label 1800 4250 0    50   ~ 0
 PWM
-$Comp
-L Connector:Screw_Terminal_01x05 J2
-U 1 1 60E6A52C
-P 1600 4450
-F 0 "J2" H 1518 4117 50  0000 C CNN
-F 1 "Screw_Terminal_01x05" H 1518 4116 50  0001 C CNN
-F 2 "" H 1600 4450 50  0001 C CNN
-F 3 "~" H 1600 4450 50  0001 C CNN
-	1    1600 4450
-	-1   0    0    1
-$EndComp
 Wire Wire Line
 	1800 4550 2200 4550
-Connection ~ 1800 4550
 Wire Wire Line
 	1800 4450 2000 4450
 Wire Wire Line
 	2850 4450 2850 4550
-Connection ~ 1800 4450
 $Comp
 L Device:R R6
@@
 Connection ~ 2000 4450
 Wire Wire Line
-	2000 4450 2850 4450
+	2000 4450 2200 4450
 Wire Wire Line
 	2200 4550 2200 4850
@@
 Wire Notes Line
 	4500 500  4500 6000
+$Comp
+L Connector:Screw_Terminal_01x06 J2
+U 1 1 60F48939
+P 1600 4450
+F 0 "J2" H 1518 4017 50  0000 C CNN
+F 1 "Screw_Terminal_01x06" H 1518 4016 50  0001 C CNN
+F 2 "" H 1600 4450 50  0001 C CNN
+F 3 "~" H 1600 4450 50  0001 C CNN
+	1    1600 4450
+	-1   0    0    1
+$EndComp
+Connection ~ 1800 4550
+Connection ~ 1800 4450
+Text Label 1800 4150 0    50   ~ 0
+TEMP
+$Comp
+L power:PWR_FLAG #FLG0101
+U 1 1 60F570D1
+P 2200 4450
+F 0 "#FLG0101" H 2200 4525 50  0001 C CNN
+F 1 "PWR_FLAG" H 2400 4500 50  0000 C CNN
+F 2 "" H 2200 4450 50  0001 C CNN
+F 3 "~" H 2200 4450 50  0001 C CNN
+	1    2200 4450
+	1    0    0    -1
+$EndComp
+Connection ~ 2200 4450
+Wire Wire Line
+	2200 4450 2850 4450
+$Comp
+L power:PWR_FLAG #FLG0102
+U 1 1 60F58B2D
+P 2200 4550
+F 0 "#FLG0102" H 2200 4625 50  0001 C CNN
+F 1 "PWR_FLAG" H 2400 4600 50  0000 C CNN
+F 2 "" H 2200 4550 50  0001 C CNN
+F 3 "~" H 2200 4550 50  0001 C CNN
+	1    2200 4550
+	1    0    0    -1
+$EndComp
+Wire Wire Line
+	9200 1250 9200 1300
+Wire Wire Line
+	9200 1600 9200 1650
+Connection ~ 9200 1650
+$Comp
+L power:PWR_FLAG #FLG0103
+U 1 1 60F663E5
+P 9200 1650
+F 0 "#FLG0103" H 9200 1725 50  0001 C CNN
+F 1 "PWR_FLAG" V 9150 1950 50  0000 C CNN
+F 2 "" H 9200 1650 50  0001 C CNN
+F 3 "~" H 9200 1650 50  0001 C CNN
+	1    9200 1650
+	0    1    1    0
+$EndComp
 $EndSCHEMATC

Commit message: footprints
Parts:
- removed C3, C4: 10uF, symbol Device:C
- removed J1: FAN, symbol Connector:Screw_Terminal_01x03
- added C3, C4: 10uF, Capacitor_THT:CP_Radial_Tantal_D5.0mm_P2.50mm, symbol Device:CP
- added J1: FAN, TerminalBlock:TerminalBlock_bornier-4_P5.08mm, symbol Connector:Screw_Terminal_01x04
- C1: footprint (none) -> Capacitor_THT:C_Disc_D4.7mm_W2.5mm_P5.00mm
- C2: value 0.1uF 50V -> 10nF; footprint (none) -> Capacitor_THT:C_Disc_D4.7mm_W2.5mm_P5.00mm
- D4, D5: footprint (none) -> Diode_THT:D_DO-35_SOD27_P7.62mm_Horizontal
- J2: footprint (none) -> TerminalBlock:TerminalBlock_bornier-6_P5.08mm
- M2: footprint (none) -> Connector_Molex:Molex_KK-254_AE-6410-04A_1x04_P2.54mm_Vertical
- R1, R2, R3, R4, R5, R6, R7: footprint (none) -> Resistor_THT:R_Axial_DIN0207_L6.3mm_D2.5mm_P7.62mm_Horizontal
Connections:
- net +12V: now also C4.1, J1.1 (Pin_1)
- net +3V3: now also C3.1
- net GND: now also C3.2, C4.2
- net TACI: now also J1.3 (Pin_3)
- net at M1.3 (-), M2.1 (-), Q2.1 (D)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: now also J1.2 (Pin_2)
- no-connect marks 1 -> 2
Changed lines of the file:
@@
 F 0 "R1" V 1293 1750 50  0000 C CNN
 F 1 "1M" V 1384 1750 50  0000 C CNN
-F 2 "" V 1430 1750 50  0001 C CNN
+F 2 "Resistor_THT:R_Axial_DIN0207_L6.3mm_D2.5mm_P7.62mm_Horizontal" V 1430 1750 50  0001 C CNN
 F 3 "~" H 1500 1750 50  0001 C CNN
 	1    1500 1750
@@
 F 0 "R3" H 2050 2000 50  0000 L CNN
 F 1 "100k" H 1950 1900 50  0000 L CNN
-F 2 "" V 2130 1950 50  0001 C CNN
+F 2 "Resistor_THT:R_Axial_DIN0207_L6.3mm_D2.5mm_P7.62mm_Horizontal" V 2130 1950 50  0001 C CNN
 F 3 "~" H 2200 1950 50  0001 C CNN
 	1    2200 1950
@@
 F 0 "R2" V 1293 2450 50  0000 C CNN
 F 1 "1M" V 1384 2450 50  0000 C CNN
-F 2 "" V 1430 2450 50  0001 C CNN
+F 2 "Resistor_THT:R_Axial_DIN0207_L6.3mm_D2.5mm_P7.62mm_Horizontal" V 1430 2450 50  0001 C CNN
 F 3 "~" H 1500 2450 50  0001 C CNN
 	1    1500 2450
@@
 F 0 "R4" H 6320 1846 50  0000 L CNN
 F 1 "1k" H 6320 1755 50  0000 L CNN
-F 2 "" V 6180 1800 50  0001 C CNN
+F 2 "Resistor_THT:R_Axial_DIN0207_L6.3mm_D2.5mm_P7.62mm_Horizontal" V 6180 1800 50  0001 C CNN
 F 3 "~" H 6250 1800 50  0001 C CNN
 	1    6250 1800
@@
 F 0 "C1" H 6365 2146 50  0000 L CNN
 F 1 "0.1uF 50V" H 6365 2055 50  0000 L CNN
-F 2 "" H 6288 1950 50  0001 C CNN
+F 2 "Capacitor_THT:C_Disc_D4.7mm_W2.5mm_P5.00mm" H 6288 1950 50  0001 C CNN
 F 3 "~" H 6250 2100 50  0001 C CNN
 	1    6250 2100
@@
 P 8950 2000
 F 0 "C2" H 8850 1900 50  0000 L CNN
-F 1 "0.1uF 50V" H 8550 1800 50  0000 L CNN
-F 2 "" H 8988 1850 50  0001 C CNN
+F 1 "10nF" H 8750 1800 50  0000 L CNN
+F 2 "Capacitor_THT:C_Disc_D4.7mm_W2.5mm_P5.00mm" H 8988 1850 50  0001 C CNN
 F 3 "~" H 8950 2000 50  0001 C CNN
 	1    8950 2000
@@
 F 0 "R5" H 9270 1496 50  0000 L CNN
 F 1 "0" H 9270 1405 50  0000 L CNN
-F 2 "" V 9130 1450 50  0001 C CNN
+F 2 "Resistor_THT:R_Axial_DIN0207_L6.3mm_D2.5mm_P7.62mm_Horizontal" V 9130 1450 50  0001 C CNN
 F 3 "~" H 9200 1450 50  0001 C CNN
 	1    9200 1450
@@
 F 0 "R6" H 2520 5046 50  0000 L CNN
 F 1 "470" H 2520 4955 50  0000 L CNN
-F 2 "" V 2380 5000 50  0001 C CNN
+F 2 "Resistor_THT:R_Axial_DIN0207_L6.3mm_D2.5mm_P7.62mm_Horizontal" V 2380 5000 50  0001 C CNN
 F 3 "~" H 2450 5000 50  0001 C CNN
 	1    2450 5000
@@
 F 0 "R7" H 2920 5046 50  0000 L CNN
 F 1 "47" H 2920 4955 50  0000 L CNN
-F 2 "" V 2780 5000 50  0001 C CNN
+F 2 "Resistor_THT:R_Axial_DIN0207_L6.3mm_D2.5mm_P7.62mm_Horizontal" V 2780 5000 50  0001 C CNN
 F 3 "~" H 2850 5000 50  0001 C CNN
 	1    2850 5000
@@
 F 0 "D5" V 2889 4582 50  0000 R CNN
 F 1 "3V3" V 2798 4582 50  0000 R CNN
-F 2 "" H 2850 4700 50  0001 C CNN
+F 2 "Diode_THT:D_DO-35_SOD27_P7.62mm_Horizontal" H 2850 4700 50  0001 C CNN
 F 3 "~" H 2850 4700 50  0001 C CNN
 	1    2850 4700
@@
 F 0 "D4" V 2489 4582 50  0000 R CNN
 F 1 "12V" V 2398 4582 50  0000 R CNN
-F 2 "" H 2450 4700 50  0001 C CNN
+F 2 "Diode_THT:D_DO-35_SOD27_P7.62mm_Horizontal" H 2450 4700 50  0001 C CNN
 F 3 "~" H 2450 4700 50  0001 C CNN
 	1    2450 4700
@@
 F 0 "M2" H 3600 1650 50  0000 L CNN
 F 1 "FAN" H 3850 1250 50  0001 L CNN
-F 2 "" H 3800 1410 50  0001 C CNN
+F 2 "Connector_Molex:Molex_KK-254_AE-6410-04A_1x04_P2.54mm_Vertical" H 3800 1410 50  0001 C CNN
 F 3 "http://www.formfactors.org/developer%5Cspecs%5Crev1_2_public.pdf" H 3800 1410 50  0001 C CNN
 	1    3800 1400
@@
 Wire Wire Line
 	3800 950  3800 1100
-$Comp
-L Connector:Screw_Terminal_01x03 J1
-U 1 1 60EB1468
-P 4400 1350
-F 0 "J1" H 4350 1600 50  0000 L CNN
-F 1 "FAN" H 4250 1100 50  0000 L CNN
-F 2 "" H 4400 1350 50  0001 C CNN
-F 3 "~" H 4400 1350 50  0001 C CNN
-	1    4400 1350
-	1    0    0    -1
-$EndComp
-Wire Wire Line
-	4200 1450 4200 1650
-Wire Wire Line
-	4200 1650 3800 1650
-Connection ~ 3800 1650
-Wire Wire Line
-	3800 950  4050 950
-Wire Wire Line
-	4050 950  4050 1350
-Wire Wire Line
-	4050 1350 4200 1350
 Connection ~ 3800 950
-Text Label 4200 1250 2    50   ~ 0
+Text Label 4200 1450 2    50   ~ 0
 TACI
 Text Label 2500 1300 2    50   ~ 0
@@
 Wire Wire Line
 	3400 1300 3500 1300
-$Comp
-L Device:C C4
-U 1 1 60EDE802
-P 2200 5000
-F 0 "C4" H 2200 5100 50  0000 L CNN
-F 1 "10uF" H 2200 4900 50  0000 L CNN
-F 2 "" H 2238 4850 50  0001 C CNN
-F 3 "~" H 2200 5000 50  0001 C CNN
-	1    2200 5000
-	1    0    0    -1
-$EndComp
-$Comp
-L Device:C C3
-U 1 1 60EDEB6F
-P 2000 5000
-F 0 "C3" H 2000 5100 50  0000 L CNN
-F 1 "10uF" H 2000 4900 50  0000 L CNN
-F 2 "" H 2038 4850 50  0001 C CNN
-F 3 "~" H 2000 5000 50  0001 C CNN
-	1    2000 5000
-	1    0    0    -1
-$EndComp
 Wire Wire Line
 	2000 4850 2000 4450
@@
 Wire Wire Line
 	1800 4650 1800 5150
-Wire Wire Line
-	1800 5150 2000 5150
-Connection ~ 2000 5150
-Wire Wire Line
-	2000 5150 2200 5150
-Connection ~ 2200 5150
 Connection ~ 2450 5150
 Wire Wire Line
@@
 $EndComp
 Connection ~ 1800 5150
-Wire Wire Line
-	2200 5150 2450 5150
 Wire Notes Line
 	7500 500  7500 3500
@@
 F 0 "J2" H 1518 4017 50  0000 C CNN
 F 1 "Screw_Terminal_01x06" H 1518 4016 50  0001 C CNN
-F 2 "" H 1600 4450 50  0001 C CNN
+F 2 "TerminalBlock:TerminalBlock_bornier-6_P5.08mm" H 1600 4450 50  0001 C CNN
 F 3 "~" H 1600 4450 50  0001 C CNN
 	1    1600 4450
@@
 	0    1    1    0
 $EndComp
+Wire Wire Line
+	1800 5150 2000 5150
+$Comp
+L Device:CP C3
+U 1 1 60F7DF0B
+P 2000 5000
+F 0 "C3" H 2000 5100 50  0000 L CNN
+F 1 "10uF" H 2000 4900 50  0000 L CNN
+F 2 "Capacitor_THT:CP_Radial_Tantal_D5.0mm_P2.50mm" H 2038 4850 50  0001 C CNN
+F 3 "~" H 2000 5000 50  0001 C CNN
+	1    2000 5000
+	1    0    0    -1
+$EndComp
+Connection ~ 2000 5150
+Wire Wire Line
+	2000 5150 2200 5150
+Connection ~ 2200 5150
+Wire Wire Line
+	2200 5150 2450 5150
+$Comp
+L Device:CP C4
+U 1 1 60F815A6
+P 2200 5000
+F 0 "C4" H 2200 5100 50  0000 L CNN
+F 1 "10uF" H 2200 4900 50  0000 L CNN
+F 2 "Capacitor_THT:CP_Radial_Tantal_D5.0mm_P2.50mm" H 2238 4850 50  0001 C CNN
+F 3 "~" H 2200 5000 50  0001 C CNN
+	1    2200 5000
+	1    0    0    -1
+$EndComp
+$Comp
+L Connector:Screw_Terminal_01x04 J1
+U 1 1 60F8B616
+P 4400 1350
+F 0 "J1" H 4350 1550 50  0000 L CNN
+F 1 "FAN" H 4300 1050 50  0000 L CNN
+F 2 "TerminalBlock:TerminalBlock_bornier-4_P5.08mm" H 4400 1350 50  0001 C CNN
+F 3 "~" H 4400 1350 50  0001 C CNN
+	1    4400 1350
+	1    0    0    -1
+$EndComp
+NoConn ~ 4200 1550
+Wire Wire Line
+	4200 950  4200 1250
+Wire Wire Line
+	3800 950  4200 950
+Wire Wire Line
+	3800 1650 3950 1650
+Wire Wire Line
+	3950 1650 3950 1350
+Wire Wire Line
+	3950 1350 4200 1350
+Connection ~ 3800 1650
 $EndSCHEMATC

Commit message: pcb layout
Parts:
- added R8: 1k, Resistor_THT:R_Axial_DIN0207_L6.3mm_D2.5mm_P7.62mm_Horizontal, symbol Device:R
- D4, D5: footprint Diode_THT:D_DO-35_SOD27_P7.62mm_Horizontal -> LED_THT:LED_D5.0mm
Connections:
- net +3V3: now also R8.1; no longer Q4.1 (D)
- new net: Q4.1 (D), R8.2
Changed lines of the file:
@@
 L power:+3.3V #PWR03
 U 1 1 60EA8063
-P 5550 1400
-F 0 "#PWR03" H 5550 1250 50  0001 C CNN
-F 1 "+3.3V" H 5565 1573 50  0000 C CNN
-F 2 "" H 5550 1400 50  0001 C CNN
-F 3 "" H 5550 1400 50  0001 C CNN
-	1    5550 1400
-	1    0    0    -1
-$EndComp
-Wire Wire Line
-	5550 1400 5550 1750
+P 5550 1450
+F 0 "#PWR03" H 5550 1300 50  0001 C CNN
+F 1 "+3.3V" H 5565 1623 50  0000 C CNN
+F 2 "" H 5550 1450 50  0001 C CNN
+F 3 "" H 5550 1450 50  0001 C CNN
+	1    5550 1450
+	1    0    0    -1
+$EndComp
 Text Label 5550 2600 2    50   ~ 0
 TACO
@@
 F 0 "D5" V 2889 4582 50  0000 R CNN
 F 1 "3V3" V 2798 4582 50  0000 R CNN
-F 2 "Diode_THT:D_DO-35_SOD27_P7.62mm_Horizontal" H 2850 4700 50  0001 C CNN
+F 2 "LED_THT:LED_D5.0mm" H 2850 4700 50  0001 C CNN
 F 3 "~" H 2850 4700 50  0001 C CNN
 	1    2850 4700
@@
 F 0 "D4" V 2489 4582 50  0000 R CNN
 F 1 "12V" V 2398 4582 50  0000 R CNN
-F 2 "Diode_THT:D_DO-35_SOD27_P7.62mm_Horizontal" H 2450 4700 50  0001 C CNN
+F 2 "LED_THT:LED_D5.0mm" H 2450 4700 50  0001 C CNN
 F 3 "~" H 2450 4700 50  0001 C CNN
 	1    2450 4700
@@
 	3950 1350 4200 1350
 Connection ~ 3800 1650
+$Comp
+L Device:R R8
+U 1 1 6102866A
+P 5550 1600
+F 0 "R8" H 5620 1646 50  0000 L CNN
+F 1 "1k" H 5620 1555 50  0000 L CNN
+F 2 "Resistor_THT:R_Axial_DIN0207_L6.3mm_D2.5mm_P7.62mm_Horizontal" V 5480 1600 50  0001 C CNN
+F 3 "~" H 5550 1600 50  0001 C CNN
+	1    5550 1600
+	1    0    0    -1
+$EndComp
 $EndSCHEMATC

Commit message: layout done
Parts:
- R5: value 0 -> 1K
- R6: value 470 -> 560
- R7: value 47 -> 56
Connections:
- net FAN-: now reaches J1.2 (Pin_2), M1.3 (-), M2.1 (-), Q2.1 (D), Q3.1 (D)
Other:
- note added: "5mm Green LED\nVf = 2.181V @ 19.52 mA +1.6°C"
Changed lines of the file:
@@
 P 9200 1450
 F 0 "R5" H 9270 1496 50  0000 L CNN
-F 1 "0" H 9270 1405 50  0000 L CNN
+F 1 "1K" H 9270 1405 50  0000 L CNN
 F 2 "Resistor_THT:R_Axial_DIN0207_L6.3mm_D2.5mm_P7.62mm_Horizontal" V 9130 1450 50  0001 C CNN
 F 3 "~" H 9200 1450 50  0001 C CNN
@@
 P 2450 5000
 F 0 "R6" H 2520 5046 50  0000 L CNN
-F 1 "470" H 2520 4955 50  0000 L CNN
+F 1 "560" H 2520 4955 50  0000 L CNN
 F 2 "Resistor_THT:R_Axial_DIN0207_L6.3mm_D2.5mm_P7.62mm_Horizontal" V 2380 5000 50  0001 C CNN
 F 3 "~" H 2450 5000 50  0001 C CNN
@@
 P 2850 5000
 F 0 "R7" H 2920 5046 50  0000 L CNN
-F 1 "47" H 2920 4955 50  0000 L CNN
+F 1 "56" H 2920 4955 50  0000 L CNN
 F 2 "Resistor_THT:R_Axial_DIN0207_L6.3mm_D2.5mm_P7.62mm_Horizontal" V 2780 5000 50  0001 C CNN
 F 3 "~" H 2850 5000 50  0001 C CNN
@@
 	1    0    0    -1
 $EndComp
+Text Label 2950 1650 2    50   ~ 0
+FAN-
+Text Notes 3050 4350 0    50   ~ 0
+5mm Green LED\nVf = 2.181V @ 19.52 mA +1.6°C
 $EndSCHEMATC

Commit message: schematic and silkscreen nits
Parts:
- R4, R8: value 1k -> 1K
Changed lines of the file:
@@
 Text Notes 3000 2400 0    50   ~ 0
 Two MOSFETs for more current.
-Text Notes 550  650  0    50   ~ 0
-60 Hz PWM
 $Comp
 L Device:R R2
@@
 P 6250 1800
 F 0 "R4" H 6320 1846 50  0000 L CNN
-F 1 "1k" H 6320 1755 50  0000 L CNN
+F 1 "1K" H 6320 1755 50  0000 L CNN
 F 2 "Resistor_THT:R_Axial_DIN0207_L6.3mm_D2.5mm_P7.62mm_Horizontal" V 6180 1800 50  0001 C CNN
 F 3 "~" H 6250 1800 50  0001 C CNN
@@
 P 5550 1600
 F 0 "R8" H 5620 1646 50  0000 L CNN
-F 1 "1k" H 5620 1555 50  0000 L CNN
+F 1 "1K" H 5620 1555 50  0000 L CNN
 F 2 "Resistor_THT:R_Axial_DIN0207_L6.3mm_D2.5mm_P7.62mm_Horizontal" V 5480 1600 50  0001 C CNN
 F 3 "~" H 5550 1600 50  0001 C CNN
@@
 Text Label 2950 1650 2    50   ~ 0
 FAN-
+Text Notes 550  650  0    50   ~ 0
+60 Hz PWM
 Text Notes 3050 4350 0    50   ~ 0
 5mm Green LED\nVf = 2.181V @ 19.52 mA +1.6°C
