File: hw/fanctl.sch (KiCad schematic (older format))
At the start: 26 parts, among them J1 FAN, J2 Screw_Terminal_01x06, M1 FAN, M2 FAN, Q1 BS170, Q2 BS170, Q3 BS170, Q4 BS170, U1 MCP9700-E

Commit message: kicad 5.1
Parts:
- U1: symbol synack-common:MCP9700-E -> fanctl-rescue:MCP9700-E-synack-common
Other:
- moved on the sheet: C2, R5
Changed lines of the file:
@@
 EELAYER 30 0
 EELAYER END
-$Descr A4 11693 8268
+$Descr USLetter 11000 8500
 encoding utf-8
 Sheet 1 1
@@
 	900  2600 1600 2600
 $Comp
-L synack-common:MCP9700-E U1
+L fanctl-rescue:MCP9700-E-synack-common U1
 U 1 1 60FA1D0F
-P 9200 2000
-F 0 "U1" H 9550 2300 50  0000 R CNN
-F 1 "MCP9700-E" H 9700 1700 50  0000 R CNN
-F 2 "Package_TO_SOT_THT:TO-92_Inline" H 10200 1850 50  0001 C CNN
-F 3 "https://ww1.microchip.com/downloads/en/DeviceDoc/20001942G.pdf" H 9200 2000 50  0001 C CNN
-	1    9200 2000
-	1    0    0    -1
-$EndComp
-Text Label 9650 2000 0    50   ~ 0
+P 8950 2050
+F 0 "U1" H 9300 2350 50  0000 R CNN
+F 1 "MCP9700-E" H 9450 1750 50  0000 R CNN
+F 2 "Package_TO_SOT_THT:TO-92_Inline" H 9950 1900 50  0001 C CNN
+F 3 "https://ww1.microchip.com/downloads/en/DeviceDoc/20001942G.pdf" H 8950 2050 50  0001 C CNN
+	1    8950 2050
+	1    0    0    -1
+$EndComp
+Text Label 9400 2050 0    50   ~ 0
 TEMP
 $Comp
 L Device:C C2
 U 1 1 60FA9761
-P 8950 2000
-F 0 "C2" H 8850 1900 50  0000 L CNN
-F 1 "10nF" H 8750 1800 50  0000 L CNN
-F 2 "Capacitor_THT:C_Disc_D4.7mm_W2.5mm_P5.00mm" H 8988 1850 50  0001 C CNN
-F 3 "~" H 8950 2000 50  0001 C CNN
-	1    8950 2000
-	1    0    0    -1
-$EndComp
-Wire Wire Line
-	8950 1850 8950 1650
-Wire Wire Line
-	8950 1650 9200 1650
-Wire Wire Line
-	8950 2150 8950 2350
-Wire Wire Line
-	8950 2350 9200 2350
+P 8700 2050
+F 0 "C2" H 8600 1950 50  0000 L CNN
+F 1 "10nF" H 8500 1850 50  0000 L CNN
+F 2 "Capacitor_THT:C_Disc_D4.7mm_W2.5mm_P5.00mm" H 8738 1900 50  0001 C CNN
+F 3 "~" H 8700 2050 50  0001 C CNN
+	1    8700 2050
+	1    0    0    -1
+$EndComp
+Wire Wire Line
+	8700 1900 8700 1700
+Wire Wire Line
+	8700 1700 8950 1700
+Wire Wire Line
+	8700 2200 8700 2400
+Wire Wire Line
+	8700 2400 8950 2400
 $Comp
 L power:+3.3V #PWR06
 U 1 1 60FB0DF1
-P 9200 1250
-F 0 "#PWR06" H 9200 1100 50  0001 C CNN
-F 1 "+3.3V" H 9215 1423 50  0000 C CNN
-F 2 "" H 9200 1250 50  0001 C CNN
-F 3 "" H 9200 1250 50  0001 C CNN
-	1    9200 1250
+P 8950 1300
+F 0 "#PWR06" H 8950 1150 50  0001 C CNN
+F 1 "+3.3V" H 8965 1473 50  0000 C CNN
+F 2 "" H 8950 1300 50  0001 C CNN
+F 3 "" H 8950 1300 50  0001 C CNN
+	1    8950 1300
 	1    0    0    -1
 $EndComp
@@
 L power:GND #PWR07
 U 1 1 60FB15C2
-P 9200 2350
-F 0 "#PWR07" H 9200 2100 50  0001 C CNN
-F 1 "GND" H 9205 2177 50  0000 C CNN
-F 2 "" H 9200 2350 50  0001 C CNN
-F 3 "" H 9200 2350 50  0001 C CNN
-	1    9200 2350
-	1    0    0    -1
-$EndComp
-Connection ~ 9200 2350
+P 8950 2400
+F 0 "#PWR07" H 8950 2150 50  0001 C CNN
+F 1 "GND" H 8955 2227 50  0000 C CNN
+F 2 "" H 8950 2400 50  0001 C CNN
+F 3 "" H 8950 2400 50  0001 C CNN
+	1    8950 2400
+	1    0    0    -1
+$EndComp
+Connection ~ 8950 2400
 $Comp
 L Device:R R5
 U 1 1 60FB1FE4
-P 9200 1450
-F 0 "R5" H 9270 1496 50  0000 L CNN
-F 1 "1K" H 9270 1405 50  0000 L CNN
-F 2 "Resistor_THT:R_Axial_DIN0207_L6.3mm_D2.5mm_P7.62mm_Horizontal" V 9130 1450 50  0001 C CNN
-F 3 "~" H 9200 1450 50  0001 C CNN
-	1    9200 1450
+P 8950 1500
+F 0 "R5" H 9020 1546 50  0000 L CNN
+F 1 "1K" H 9020 1455 50  0000 L CNN
+F 2 "Resistor_THT:R_Axial_DIN0207_L6.3mm_D2.5mm_P7.62mm_Horizontal" V 8880 1500 50  0001 C CNN
+F 3 "~" H 8950 1500 50  0001 C CNN
+	1    8950 1500
 	1    0    0    -1
 $EndComp
 Text Notes 7550 600  0    50   ~ 0
 Adjust RC values to filter digital noise
-Wire Notes Line
-	500  3500 11200 3500
 $Comp
 L power:+12V #PWR09
@@
 $EndComp
 Wire Wire Line
-	9200 1250 9200 1300
-Wire Wire Line
-	9200 1600 9200 1650
-Connection ~ 9200 1650
+	8950 1300 8950 1350
+Wire Wire Line
+	8950 1650 8950 1700
+Connection ~ 8950 1700
 $Comp
 L power:PWR_FLAG #FLG0103
 U 1 1 60F663E5
-P 9200 1650
-F 0 "#FLG0103" H 9200 1725 50  0001 C CNN
-F 1 "PWR_FLAG" V 9150 1950 50  0000 C CNN
-F 2 "" H 9200 1650 50  0001 C CNN
-F 3 "~" H 9200 1650 50  0001 C CNN
-	1    9200 1650
+P 8950 1700
+F 0 "#FLG0103" H 8950 1775 50  0001 C CNN
+F 1 "PWR_FLAG" V 8900 2000 50  0000 C CNN
+F 2 "" H 8950 1700 50  0001 C CNN
+F 3 "~" H 8950 1700 50  0001 C CNN
+	1    8950 1700
 	0    1    1    0
 $EndComp
@@
 Text Notes 3050 4350 0    50   ~ 0
 5mm Green LED\nVf = 2.181V @ 19.52 mA +1.6°C
+Wire Notes Line
+	500  3500 10500 3500
 $EndSCHEMATC
